File: hardware/mark-two/boot.sch (KiCad schematic (older format))
At the start: 6 parts, among them SW1 CAS-220TA, U2 MX6UL-VM

Commit message: add USB armory Mk II rev. γ
Parts:
- U2: Mfg PN (none) -> MCIMX6Z0DVM09AB
Changed lines of the file:
@@
 EESchema Schematic File Version 4
-LIBS:armory-cache
 EELAYER 30 0
 EELAYER END
@@
 encoding utf-8
 Sheet 6 13
-Title "USB ARMORY"
-Date "2019-06-25"
-Rev "MARK II"
+Title "USB armory Mk II"
+Date "2021-02-18"
+Rev "γ"
 Comp "F-Secure"
-Comment1 "Copyright © 2019 F-Secure"
-Comment2 "License: CERN OHL v1.2"
-Comment3 "https://github.com/inversepath/usbarmory"
+Comment1 "Copyright © F-Secure Corporation"
+Comment2 "License: CERN-OHL-S"
+Comment3 "https://github.com/f-secure-foundry/usbarmory"
 Comment4 ""
 $EndDescr
@@
 F 2 "armory-kicad:SOT1534-2" H 4960 3090 60  0001 C CNN
 F 3 "https://www.nxp.com/docs/en/data-sheet/IMX6ULCEC.pdf" H 4960 3090 60  0001 C CNN
+F 4 "MCIMX6Z0DVM09AB" H 4450 4250 50  0001 C CNN "Mfg PN"
 	7    4450 4250
 	1    0    0    -1
