File: hardware/mark-two/microsd.sch (KiCad schematic (older format))
At the start: 11 parts, among them J1 microSD slot, U12 TPD6F003, U2 MX6UL-VM, U20 TPD1E10B06, U21 TPD1E10B06

Commit message: add USB armory Mk II rev. γ
Parts:
- removed U12: TPD6F003, armory-kicad:WSON-12, symbol Power_Protection:TPD6F003
- added U12: PUSB3TB6, armory-kicad:SOT1358-1, symbol armory-mkII:PUSB3TB6
- U2: Mfg PN (none) -> MCIMX6Z0DVM09AB
- U20, U21: Alternative PN (none) -> TPD1E10B06-Q1, TPD1E10B09, TPD1E10B09-Q1
Connections:
- net labels added: SD_3V3_1V8
- net labels removed: SD1_CLK_ESD, SD1_CMD_ESD, SD1_DATA0_ESD, SD1_DATA1_ESD, SD1_DATA2_ESD, SD1_DATA3_ESD
- wire segments 67 -> 64
Other:
- moved on the sheet: C105, C106, J1, R55, R56, U20, U21
