File: hardware/mark-two/power.sch (KiCad schematic (older format))
At the start: 20 parts, among them U2 MX6UL-VM

Commit message: add USB armory Mk II rev. γ
Parts:
- C103, C87, C98: Alternative PN (none) -> CL05A226MQ6ZUN8
Changed lines of the file:
@@
 EESchema Schematic File Version 4
-LIBS:armory-cache
 EELAYER 30 0
 EELAYER END
@@
 encoding utf-8
 Sheet 8 13
-Title "USB ARMORY"
-Date "2019-06-25"
-Rev "MARK II"
+Title "USB armory Mk II"
+Date "2021-02-18"
+Rev "γ"
 Comp "F-Secure"
-Comment1 "Copyright © 2019 F-Secure"
-Comment2 "License: CERN OHL v1.2"
-Comment3 "https://github.com/inversepath/usbarmory"
+Comment1 "Copyright © F-Secure Corporation"
+Comment2 "License: CERN-OHL-S"
+Comment3 "https://github.com/f-secure-foundry/usbarmory"
 Comment4 ""
 $EndDescr
@@
 F 9 "0402" H 4700 3800 30  0000 C CNN "FP"
 F 10 "6.3V/20%" H 4850 3650 30  0000 C CNN "Rating"
+F 11 "CL05A226MQ6ZUN8" H 4700 3800 50  0001 C CNN "Alternative PN"
 	1    4700 3800
 	1    0    0    -1
@@
 F 9 "0402" H 13100 4150 30  0000 C CNN "FP"
 F 10 "6.3V/20%" H 13250 4000 30  0000 C CNN "Rating"
+F 11 "CL05A226MQ6ZUN8" H 13100 4150 50  0001 C CNN "Alternative PN"
 	1    13100 4150
 	1    0    0    -1
@@
 F 9 "0402" H 11600 4150 30  0000 C CNN "FP"
 F 10 "6.3V/20%" H 11750 4000 30  0000 C CNN "Rating"
+F 11 "CL05A226MQ6ZUN8" H 11600 4150 50  0001 C CNN "Alternative PN"
 	1    11600 4150
 	1    0    0    -1
