File: hardware/mark-two/secure-element.sch (KiCad schematic (older format))
At the start: 6 parts, among them U13 ATECC608A, U4 A71CH

Commit message: add USB armory Mk II rev. γ
Parts:
- removed R4: 10K, armory-kicad:SM0201, symbol Device:R
- removed U4: A71CH, armory-kicad:SOT1999-1, symbol armory-mkII:A71CH
- added U4: SE050, armory-kicad:SOT1969-1, symbol armory-mkII:SE050
- C107: DNP (none) -> DNP
- U13: value ATECC608A -> ATECC608B-DNP; symbol armory-mkII:ATECC608A -> armory-mkII:ATECC608; DNP (none) -> DNP; Mfg PN ATECC608A-MAHDA -> ATECC608B-MAHDA; Supplier PN ATECC608A-MAHDA-SCT-ND -> ATECC608B-MAHDA-SCT-ND
Connections:
- net labels added: SE050_ENA
- net labels removed: A71CH_RESET
- wire segments 38 -> 36
- no-connect marks 5 -> 13
Other:
- note added: "Optional, not mounted on retail units."
- moved on the sheet: C5, R29
