File: hardware/mark-two/usb.sch (KiCad schematic (older format))
At the start: 40 parts, among them J2 USBC-PLUG, J3 USBC-RECEPTACLE, U14 TUSB320, U15 TPD1E10B06, U16 TPD1E10B06, U17 SN74LVC1G04, U18 FSA1208, U19 TPD8E003, U2 MX6UL-VM, U5 FPF2286UCX, U6 TPD4E05U06-Q1, U7 TPD4E05U06-Q1, U8 NX5P3090, U9 FUSB303

Commit message: add USB armory Mk II rev. γ
Parts:
- removed J2: USBC-PLUG, armory-kicad:WURTH_632712000011, symbol armory-mkII:USBC-PLUG
- added J2: USBC-PLUG_24_PIN, armory-kicad:WURTH_632712000112, symbol armory-mkII:USBC-PLUG_24_PIN
- C49, C50: Alternative PN (none) -> CL03A105KP3NSNC
- C6: Mfg PN GRM033R6YA104KE14D -> GRM033R61A104ME15D
- U14: Alternative PN (none) -> TUSB320RWBR
- U15, U16: Alternative PN (none) -> TPD1E10B06-Q1, TPD1E10B09, TPD1E10B09-Q1
- U2: Mfg PN (none) -> MCIMX6Z0DVM09AB
- U5: Alternative PN (none) -> KTS1670EUN-TR, KTS1671EUN-TR
- U6, U7: value TPD4E05U06-Q1 -> TPD4E05U06; Alternative PN (none) -> TPD4E05U06QDQARQ1
Connections:
- no-connect marks 20 -> 22
Changed lines of the file:
@@
 EESchema Schematic File Version 4
-LIBS:armory-cache
 EELAYER 30 0
 EELAYER END
@@
 encoding utf-8
 Sheet 5 13
-Title "USB ARMORY"
-Date "2019-06-25"
-Rev "MARK II"
+Title "USB armory Mk II"
+Date "2021-02-18"
+Rev "γ"
 Comp "F-Secure"
-Comment1 "Copyright © 2019 F-Secure"
-Comment2 "License: CERN OHL v1.2"
-Comment3 "https://github.com/inversepath/usbarmory"
+Comment1 "Copyright © F-Secure Corporation"
+Comment2 "License: CERN-OHL-S"
+Comment3 "https://github.com/f-secure-foundry/usbarmory"
 Comment4 ""
 $EndDescr
@@
 F 2 "armory-kicad:SOT1534-2" H 3460 240 60  0001 C CNN
 F 3 "https://www.nxp.com/docs/en/data-sheet/IMX6ULCEC.pdf" H 3460 240 60  0001 C CNN
+F 4 "MCIMX6Z0DVM09AB" H 2950 1400 50  0001 C CNN "Mfg PN"
 	8    2950 1400
 	1    0    0    -1
@@
 P 1950 9350
 F 0 "U7" H 1950 9400 50  0000 C CNN
-F 1 "TPD4E05U06-Q1" H 1950 8700 50  0000 C CNN
+F 1 "TPD4E05U06" H 1950 8700 50  0000 C CNN
 F 2 "armory-kicad:DQA-USON-10" H 1950 9350 50  0001 C CNN
 F 3 "http://www.ti.com/lit/ds/symlink/tpd6e05u06.pdf" H 1950 9350 50  0001 C CNN
@@
 F 7 "Digikey" H 1950 9350 50  0001 C CNN "Supplier"
 F 8 "296-35765-2-ND" H 1950 9350 50  0001 C CNN "Supplier PN"
+F 9 "TPD4E05U06QDQARQ1" H 1950 9350 50  0001 C CNN "Alternative PN"
 	1    1950 9350
 	1    0    0    -1
@@
 F 7 "Digikey" H 1950 9050 50  0001 C CNN "Supplier"
 F 8 "296-30406-1-ND" H 1950 9050 50  0001 C CNN "Supplier PN"
+F 9 "TPD1E10B06-Q1, TPD1E10B09, TPD1E10B09-Q1" H 1950 9050 50  0001 C CNN "Alternative PN"
 	1    1950 9050
 	1    0    0    1
@@
 F 7 "Digikey" H 4900 9050 50  0001 C CNN "Supplier"
 F 8 "296-30406-1-ND" H 4900 9050 50  0001 C CNN "Supplier PN"
+F 9 "TPD1E10B06-Q1, TPD1E10B09, TPD1E10B09-Q1" H 4900 9050 50  0001 C CNN "Alternative PN"
 	1    4900 9050
 	1    0    0    1
@@
 	13500 3200 13450 3200
 NoConn ~ 14400 3200
-Text GLabel 14550 1600 2    50   BiDi ~ 0
+Text GLabel 14550 1600 2    50   Input ~ 0
 UART2_TX
-Text GLabel 14550 1800 2    50   BiDi ~ 0
+Text GLabel 14550 1800 2    50   Output ~ 0
 UART2_RX
-Text GLabel 14550 2200 2    50   BiDi ~ 0
+Text GLabel 14550 2200 2    50   Output ~ 0
+UART2_RTS
+Text GLabel 14550 2000 2    50   Input ~ 0
 UART2_CTS
-Text GLabel 14550 2000 2    50   BiDi ~ 0
-UART2_RTS
-Text GLabel 14550 2600 2    50   BiDi ~ 0
+Text GLabel 14550 2600 2    50   Input ~ 0
 UART4_TX
-Text GLabel 14550 2800 2    50   BiDi ~ 0
+Text GLabel 14550 2800 2    50   Output ~ 0
 UART4_RX
-Text GLabel 14550 3000 2    50   BiDi ~ 0
+Text GLabel 14550 3000 2    50   Output ~ 0
 UART5_RX
-Text GLabel 14550 2400 2    50   BiDi ~ 0
+Text GLabel 14550 2400 2    50   Input ~ 0
 UART5_TX
 Wire Wire Line
@@
 F 9 "0201" H 1550 2150 30  0000 C CNN "FP"
 F 10 "10V/20%" H 1700 2000 30  0000 C CNN "Rating"
+F 11 "CL03A105KP3NSNC" H 1550 2150 50  0001 C CNN "Alternative PN"
 	1    1550 2150
 	1    0    0    -1
@@
 F 9 "0201" H 1550 3050 30  0000 C CNN "FP"
 F 10 "10V/20%" H 1700 2900 30  0000 C CNN "Rating"
+F 11 "CL03A105KP3NSNC" H 1550 3050 50  0001 C CNN "Alternative PN"
 	1    1550 3050
 	1    0    0    -1
@@
 P 4900 9800
 F 0 "U6" H 4900 9850 50  0000 C CNN
-F 1 "TPD4E05U06-Q1" H 4900 9150 50  0000 C CNN
+F 1 "TPD4E05U06" H 4900 9150 50  0000 C CNN
 F 2 "armory-kicad:DQA-USON-10" H 4900 9800 50  0001 C CNN
 F 3 "http://www.ti.com/lit/ds/symlink/tpd6e05u06.pdf" H 4900 9800 50  0001 C CNN
@@
 F 7 "Digikey" H 4900 9800 50  0001 C CNN "Supplier"
 F 8 "296-35765-2-ND" H 4900 9800 50  0001 C CNN "Supplier PN"
+F 9 "TPD4E05U06QDQARQ1" H 4900 9800 50  0001 C CNN "Alternative PN"
 	1    4900 9800
 	1    0    0    -1
@@
 F 7 "Digikey" H 9700 1725 50  0001 C CNN "Supplier"
 F 8 "FPF2286UCXOSCT-ND" H 9700 1725 50  0001 C CNN "Supplier PN"
+F 9 "KTS1670EUN-TR, KTS1671EUN-TR" H 9700 1725 50  0001 C CNN "Alternative PN"
 	1    9700 1725
 	1    0    0    -1
@@
 F 3 "~" H 8800 2275 50  0001 C CNN
 F 4 "Murata Electronics North America" H 8800 2275 50  0001 C CNN "Mfg"
-F 5 "GRM033R6YA104KE14D" H 8800 2275 50  0001 C CNN "Mfg PN"
+F 5 "GRM033R61A104ME15D" H 8800 2275 50  0001 C CNN "Mfg PN"
 F 6 "X5R, 10%, 35V" H 8800 2275 50  0001 C CNN "Desc"
 F 7 "Digikey" H 8800 2275 50  0001 C CNN "Supplier"
@@
 Text Label 3050 4900 2    50   ~ 0
 TYPEC_B11
-$Comp
-L armory-mkII:USBC-PLUG J2
-U 1 1 5C7F9A68
-P 4850 4600
-AR Path="/5C7F9A68" Ref="J2"  Part="1"
-AR Path="/538352BD/5C7F9A68" Ref="J2"  Part="1"
-F 0 "J2" H 4850 4650 50  0000 C CNN
-F 1 "USBC-PLUG" H 4850 1950 50  0000 C CNN
-F 2 "armory-kicad:WURTH_632712000011" H 4800 4600 50  0001 C CNN
-F 3 "https://katalog.we-online.de/em/datasheet/632712000011.pdf" H 4800 4600 50  0001 C CNN
-F 4 "Würth Elektronik " H 4850 4600 50  0001 C CNN "Mfg"
-F 5 "632712000011" H 4850 4600 50  0001 C CNN "Mfg PN"
-F 6 "Type-C plug" H 4850 4600 50  0001 C CNN "Desc"
-F 7 "Digikey" H 4850 4600 50  0001 C CNN "Supplier"
-F 8 "732-9616-2-ND" H 4850 4600 50  0001 C CNN "Supplier PN"
-	1    4850 4600
-	1    0    0    -1
-$EndComp
 Wire Wire Line
 	5450 6900 5450 7200
@@
 F 7 "Digikey" H 9700 6000 50  0001 C CNN "Supplier"
 F 8 "296-42175-1-ND" H 9700 6000 50  0001 C CNN "Supplier PN"
+F 9 "TUSB320RWBR" H 9700 6000 50  0001 C CNN "Alternative PN"
 	1    9700 6000
 	1    0    0    -1
@@
 Wire Wire Line
 	8850 7100 8850 7300
+$Comp
+L armory-mkII:USBC-PLUG_24_PIN J2
+U 1 1 5FB03100
+P 4850 4600
+F 0 "J2" H 4850 4650 50  0000 C CNN
+F 1 "USBC-PLUG_24_PIN" H 4850 1950 50  0000 C CNN
+F 2 "armory-kicad:WURTH_632712000112" H 4800 4600 50  0001 C CNN
+F 3 "https://www.we-online.de/katalog/datasheet/632712000112.pdf" H 4800 4600 50  0001 C CNN
+F 4 "Würth Elektronik" H 4850 4600 50  0001 C CNN "Mfg"
+F 5 "632712000112" H 4850 4600 50  0001 C CNN "Mfg PN"
+F 6 "Type-C plug" H 4850 4600 50  0001 C CNN "Desc"
+F 7 "Digikey" H 4850 4600 50  0001 C CNN "Supplier"
+F 8 " 732-13725-ND" H 4850 4600 50  0001 C CNN "Supplier PN"
+	1    4850 4600
+	1    0    0    -1
+$EndComp
+NoConn ~ 5400 5700
+NoConn ~ 5400 5900
 $EndSCHEMATC
