File: hardware/mark-two-lan/usb.kicad_sch (KiCad schematic)
At the start: 19 parts, among them J1 USBC-RECEPTACLE, U14 TUSB320, U15 TPD1E10B06, U2 MX6UL-VM, U5 FPF2286UCX, U6 TPD4E05U06

Commit message: Fix comments
Other:
- note added: "Type-C ESD protection"
- note added: "Type-C port controller"
- note removed: "Type-C plug ESD protection"
- note removed: "Type-C plug port controller"
Changed lines of the file:
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@@
     (effects (font (size 1.27 1.27)) (justify left bottom))
   )
-  (text "Type-C plug port controller" (at 201.93 110.49 0)
+  (text "Type-C port controller" (at 201.93 110.49 0)
     (effects (font (size 2.54 2.54)) (justify left bottom))
   )
@@
     (effects (font (size 1.27 1.27)) (justify left bottom))
   )
-  (text "Type-C plug ESD protection" (at 96.52 218.44 0)
+  (text "Type-C ESD protection" (at 96.52 218.44 0)
     (effects (font (size 2.54 2.54)) (justify left bottom))
   )
